File: OBG-SVF-panelPCB/OBG-SVF-panelpcb.kicad_pcb (KiCad board)
At the start: 2 copper layers, 55.9 x 91.4 mm, 22 parts, among them J1 AudioJack2, J2 AudioJack2, J3 AudioJack2, J4 AudioJack2, J5 AudioJack2, J6 AudioJack2, J9 Conn_02x06_Odd_Even

Commit message: Panel PCB Gerbers, some schematic updates
Parts:
- moved R8 0.21 mm to (152.5, 84.0)
Connections:
- R1 pad 1: +12V -> GND
- R1 pad 3: GND -> +12V
- R31 pad 1: Net-(J1-Pad3) -> GND
- R31 pad 3: GND -> Net-(J1-Pad3)
- R32 pad 1: Net-(J3-Pad3) -> GND
- R32 pad 3: GND -> Net-(J3-Pad3)
- R33 pad 1: Net-(J5-Pad3) -> GND
- R33 pad 3: GND -> Net-(J5-Pad3)
Routing:
- net CVIn: track 56.0 -> 65.8 mm
- net Net-(R29-Pad2): track 10.6 -> 20.3 mm
- net +12V: track 20.6 -> 14.8 mm
- net Net-(R31-Pad2): track 17.1 -> 21.9 mm
- net Net-(R33-Pad2): track 21.2 -> 17.2 mm
